File: HandPICd24.kicad_pcb (KiCad board)
At the start: 4 copper layers, 100 x 100 mm, 112 parts, among them J1 Conn_02x06_Odd_Even, J10 Conn_02x14_Odd_Even, J11 Conn_02x14_Odd_Even, J12 Conn_02x14_Odd_Even, J13 Conn_02x14_Odd_Even, J14 Conn_02x14_Odd_Even, J15 Conn_02x14_Odd_Even, J16 Conn_02x14_Odd_Even, J17 Conn_02x14_Odd_Even, J18 Conn_01x06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

Commit message: Add files via upload
Parts:
- moved G102 0.51 mm to (110.5, 152.3)
Other:
- board text added: "Special thanks to: Garth Wilson @ wilsonminesco.com Bill Shen aka {dblquote}plasmo{dblquote} @ www.retrobrewcomputers.org George Foot @ github.com/gfoot BDD @ http://sbc.steggy.net/ Voja Antonic @ voja.rs Everyone @ 6502.org"
- board text removed: "Special thanks to: Garth Wilson @ wilsonminesco.com Bill Shen aka {dblquote}plasmo{dblquote} @ www.retrobrewcomputers.org BDD @ http://sbc.steggy.net/ Voja Antonic @ voja.rs Everyone @ 6502.org"
Changed lines of the file:
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@@
   )
   (footprint "JustPIC:HandPickedTitle" (layer "F.Cu")
-    (at 110.49 151.765)
+    (at 110.49 152.273)
     (attr board_only exclude_from_pos_files exclude_from_bom)
     (fp_text reference "G102" (at 0 0) (layer "F.SilkS") hide
@@
   (gr_line (start 136.525 161.925) (end 136.525 160.655)
     (stroke (width 0.15) (type default)) (layer "F.SilkS"))
+  (gr_line (start 245.5 61.95) (end 245.5 44.45)
+    (stroke (width 0.15) (type default)) (layer "F.SilkS"))
   (gr_line (start 128.905 136.398) (end 128.905 147.828)
     (stroke (width 0.15) (type default)) (layer "F.SilkS"))
@@
   (gr_line (start 125.603 141.605) (end 126.238 140.97)
     (stroke (width 0.15) (type default)) (layer "F.SilkS"))
+  (gr_line (start 190.5 61.95) (end 245.5 61.95)
+    (stroke (width 0.15) (type default)) (layer "F.SilkS"))
   (gr_line (start 129.667 134.112) (end 128.905 134.112)
     (stroke (width 0.15) (type default)) (layer "F.SilkS"))
+  (gr_line (start 245.5 44.45) (end 190.5 44.45)
+    (stroke (width 0.15) (type default)) (layer "F.SilkS"))
+  (gr_line (start 190.5 44.45) (end 190.5 61.95)
+    (stroke (width 0.15) (type default)) (layer "F.SilkS"))
   (gr_line (start 114.173 113.03) (end 112.903 113.03)
     (stroke (width 0.15) (type default)) (layer "F.SilkS"))
@@
     (effects (font (size 1 1) (thickness 0.15)) (justify left bottom mirror))
   )
-  (gr_text "Special thanks to:\nGarth Wilson @ wilsonminesco.com\nBill Shen aka {dblquote}plasmo{dblquote} \n    @ www.retrobrewcomputers.org\nBDD @ http://sbc.steggy.net/\nVoja Antonic @ voja.rs\nEveryone @ 6502.org\n" (at 126.365 127) (layer "B.SilkS")
+  (gr_text "Special thanks to:\nGarth Wilson @ wilsonminesco.com\nBill Shen aka {dblquote}plasmo{dblquote} \n    @ www.retrobrewcomputers.org\nGeorge Foot @ github.com/gfoot\nBDD @ http://sbc.steggy.net/\nVoja Antonic @ voja.rs\nEveryone @ 6502.org\n" (at 126.365 127) (layer "B.SilkS")
     (effects (font (size 1 1) (thickness 0.15)) (justify left bottom mirror))
   )
@@
   (segment (start 136.846 135.78) (end 131.127 130.061) (width 0.25) (layer "B.Cu") (net 40))
   (segment (start 136.846 155.889) (end 136.846 135.78) (width 0.25) (layer "B.Cu") (net 40))
-  (segment (start 109.9311 153.6406) (end 138.4597 153.6406) (width 0.25) (layer "F.Cu") (net 41))
   (segment (start 145.5347 158.3826) (end 145.5347 158.75) (width 0.25) (layer "F.Cu") (net 41))
+  (segment (start 143.8337 157.5747) (end 144.7268 157.5747) (width 0.25) (layer "F.Cu") (net 41))
+  (segment (start 142.9946 156.7356) (end 143.8337 157.5747) (width 0.25) (layer "F.Cu") (net 41))
+  (segment (start 144.7268 157.5747) (end 145.5347 158.3826) (width 0.25) (layer "F.Cu") (net 41))
   (segment (start 92.9473 108.2262) (end 92.9473 120.7322) (width 0.25) (layer "F.Cu") (net 41))
   (segment (start 103.378 99.0054) (end 101.5671 97.1945) (width 0.25) (layer "F.Cu") (net 41))
-  (segment (start 101.5671 97.1945) (end 100.2968 97.1945) (width 0.25) (layer "F.Cu") (net 41))
+  (segment (start 145.5347 158.75) (end 146.71 158.75) (width 0.25) (layer "F.Cu") (net 41))
   (segment (start 138.7108 153.8917) (end 141.0614 153.8917) (width 0.25) (layer "F.Cu") (net 41))
-  (segment (start 141.0614 153.8917) (end 142.9946 155.8249) (width 0.25) (layer "F.Cu") (net 41))
   (segment (start 142.9946 155.8249) (end 142.9946 156.7356) (width 0.25) (layer "F.Cu") (net 41))
-  (segment (start 144.7268 157.5747) (end 145.5347 158.3826) (width 0.25) (layer "F.Cu") (net 41))
+  (segment (start 101.5671 97.1945) (end 100.2968 97.1945) (width 0.25) (layer "F.Cu") (net 41))
+  (segment (start 109.9311 153.6406) (end 138.4597 153.6406) (width 0.25) (layer "F.Cu") (net 41))
+  (segment (start 141.0614 153.8917) (end 142.9946 155.8249) (width 0.25) (layer "F.Cu") (net 41))
+  (segment (start 138.4597 153.6406) (end 138.7108 153.8917) (width 0.25) (layer "F.Cu") (net 41))
+  (segment (start 107.3565 151.066) (end 109.9311 153.6406) (width 0.25) (layer "F.Cu") (net 41))
   (segment (start 103.378 99.0054) (end 103.378 98.425) (width 0.25) (layer "F.Cu") (net 41))
   (segment (start 96.6472 100.8441) (end 96.6472 104.5263) (width 0.25) (layer "F.Cu") (net 41))
-  (segment (start 142.9946 156.7356) (end 143.8337 157.5747) (width 0.25) (layer "F.Cu") (net 41))
   (segment (start 110.338 107.09) (end 103.378 100.13) (width 0.25) (layer "F.Cu") (net 41))
-  (segment (start 138.4597 153.6406) (end 138.7108 153.8917) (width 0.25) (layer "F.Cu") (net 41))
   (segment (start 103.378 100.13) (end 103.378 99.0054) (width 0.25) (layer "F.Cu") (net 41))
-  (segment (start 107.3565 151.066) (end 109.9311 153.6406) (width 0.25) (layer "F.Cu") (net 41))
   (segment (start 110.338 107.965) (end 110.338 107.09) (width 0.25) (layer "F.Cu") (net 41))
   (segment (start 100.2968 97.1945) (end 96.6472 100.8441) (width 0.25) (layer "F.Cu") (net 41))
-  (segment (start 143.8337 157.5747) (end 144.7268 157.5747) (width 0.25) (layer "F.Cu") (net 41))
   (segment (start 96.6472 104.5263) (end 92.9473 108.2262) (width 0.25) (layer "F.Cu") (net 41))
-  (segment (start 146.71 158.75) (end 145.5347 158.75) (width 0.25) (layer "F.Cu") (net 41))
   (via (at 92.9473 120.7322) (size 0.8) (drill 0.4) (layers "F.Cu" "B.Cu") (net 41))
   (via (at 107.3565 151.066) (size 0.8) (drill 0.4) (layers "F.Cu" "B.Cu") (net 41))
+  (segment (start 107.3565 151.066) (end 102.3405 146.05) (width 0.25) (layer "B.Cu") (net 41))
   (segment (start 92.9473 134.0359) (end 96.393 137.4816) (width 0.25) (layer "B.Cu") (net 41))
-  (segment (start 96.393 146.05) (end 102.3405 146.05) (width 0.25) (layer "B.Cu") (net 41))
-  (segment (start 102.3405 146.05) (end 107.3565 151.066) (width 0.25) (layer "B.Cu") (net 41))
   (segment (start 92.9473 120.7322) (end 92.9473 134.0359) (width 0.25) (layer "B.Cu") (net 41))
   (segment (start 96.393 137.4816) (end 96.393 146.05) (width 0.25) (layer "B.Cu") (net 41))
+  (segment (start 102.3405 146.05) (end 96.393 146.05) (width 0.25) (layer "B.Cu") (net 41))
   (segment (start 99.06 86.995) (end 96.3753 86.995) (width 0.25) (layer "F.Cu") (net 43))
   (segment (start 95.25 86.995) (end 96.3753 86.995) (width 0.25) (layer "F.Cu") (net 43))
