File: HandPICd24.kicad_sch (KiCad schematic)
At the start: 109 parts, among them J1 Conn_02x06_Odd_Even, J10 Conn_01x06, J10 Conn_02x14_Odd_Even, J11 Conn_02x14_Odd_Even, J12 Conn_02x14_Odd_Even, J13 Conn_02x14_Odd_Even, J14 Conn_02x14_Odd_Even, J15 Conn_02x14_Odd_Even, J16 Conn_02x14_Odd_Even, J17 Conn_02x14_Odd_Even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

Commit message: Add files via upload
Other:
- note added: "LED needs to be flipped!!!"
Changed lines of the file:
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@@
     (effects (font (size 1.27 1.27)) (justify left bottom))
+  )
+  (text "LED needs to be flipped!!!" (at 66.04 154.94 0)
+    (effects (font (size 2.54 2.54)) (justify left bottom))
   )
   (global_label "JOY-SELECT" (shape input) (at 170.18 143.51 270) (fields_autoplaced)
